Commit message: [fix] linkを2つに

File: b3m_description/urdf/b3m.urdf (robot description, URDF)
Before this commit: robot origins, 2 links, 1 joints
Links:
- removed link wheel
- added link wheel1; visual cylinder length=0.05 radius=0.5
- added link wheel2; visual cylinder length=0.05 radius=0.5
Joints:
- joint base_to_wheel: child wheel -> wheel2; origin xyz=0.3 0.1 0.1 -> xyz=0.6 0.1 0.1

Commit message: [fix] nodeネームとかコマンドライン引数の処理を修正

File: b3m_description/urdf/b3m.urdf (robot description, URDF)
Before this commit: robot origins, 3 links, 1 joints
Links:
- removed link wheel2
- added link wheel0; visual cylinder length=0.05 radius=0.5
Joints:
- removed joint base_to_wheel
- added joint base_to_wheel0: type continuous, parent base_link, child wheel0, origin xyz=0.3 0.1 0.1, axis 0 1 0
- added joint base_to_wheel1: type continuous, parent base_link, child wheel1, origin xyz=0.6 0.1 0.1, axis 0 1 0

Commit message: [modify] 3つめのサーボモータを使う設定を追加

File: b3m_description/urdf/b3m.urdf (robot description, URDF)
Before this commit: robot origins, 3 links, 2 joints
Links:
- added link wheel2; visual cylinder length=0.05 radius=0.5
- added link wheel3; visual cylinder length=0.05 radius=0.5
Joints:
- added joint base_to_wheel2: type continuous, parent base_link, child wheel2, origin xyz=0.6 0.1 0.1, axis 0 1 0
- added joint base_to_wheel3: type continuous, parent base_link, child wheel3, origin xyz=0.6 0.1 0.1, axis 0 1 0
